File: adapter/_autosave-ebus-pri.sch (KiCad schematic (older format))
At the start: 28 parts, among them IC1 TLC393CP, J1 Conn_02x13_Odd_Even, J3 DS18B20_IN, P3 ebus1, P4 ebus2, Q1 BC338, U1 CNY17-4, U2 CNY17-4

Commit message: ready for print
Parts:
- R5: value 4.7K -> 10k
Connections:
- net TEMP_INS: now also J1.24 (Pin_24); no longer J1.17 (Pin_17)
Changed lines of the file:
@@
 P 4850 1100
 F 0 "R5" V 4930 1100 50  0000 C CNN
-F 1 "4.7K" V 4850 1100 50  0000 C CNN
+F 1 "10k" V 4850 1100 50  0000 C CNN
 F 2 "Resistor_THT:R_Axial_DIN0204_L3.6mm_D1.6mm_P2.54mm_Vertical" V 4780 1100 50  0001 C CNN
 F 3 "" H 4850 1100 50  0001 C CNN
@@
 	1    0    0    -1
 $EndComp
-Text GLabel 3100 6350 2    60   Input ~ 0
+Text GLabel 2200 6650 0    60   Input ~ 0
 TEMP_INS
 Text GLabel 3100 5550 2    60   Input ~ 0
@@
 	2950 5850 3100 5850
 Wire Wire Line
-	2950 6350 3100 6350
-Wire Wire Line
 	8850 4050 8850 5350
+Wire Wire Line
+	2200 6650 2450 6650
 $EndSCHEMATC
