File: adapter/ebus-pri.kicad_pcb (KiCad board)
At the start: 2 copper layers, 29 parts, among them IC1 TLC393CP, J1 Conn_02x13_Odd_Even, J3 DS18B20_IN, P3 ebus1, P4 ebus2, Q1 BC338, U1 CNY17-4, U2 CNY17-4

Commit message: ready for print
Parts:
- removed R15: 0ohm, Resistor_THT:R_Axial_DIN0207_L6.3mm_D2.5mm_P7.62mm_Horizontal
- D3: footprint Diode_THT:D_DO-41_SOD81_P12.70mm_Horizontal -> Diode_THT:D_DO-41_SOD81_P2.54mm_Vertical_KathodeUp
- D4, D5, D6, D7: footprint Diode_THT:D_DO-41_SOD81_P7.62mm_Horizontal -> Diode_THT:D_DO-41_SOD81_P2.54mm_Vertical_KathodeUp
- J1: moved to B.Cu
- R11: footprint Resistor_THT:R_Axial_DIN0207_L6.3mm_D2.5mm_P10.16mm_Horizontal -> Resistor_THT:R_Axial_DIN0204_L3.6mm_D1.6mm_P2.54mm_Vertical
- R12: footprint Resistor_THT:R_Axial_DIN0309_L9.0mm_D3.2mm_P12.70mm_Horizontal -> Resistor_THT:R_Axial_DIN0207_L6.3mm_D2.5mm_P2.54mm_Vertical
- R13: footprint Resistor_THT:R_Axial_DIN0207_L6.3mm_D2.5mm_P10.16mm_Horizontal -> Resistor_THT:R_Axial_DIN0207_L6.3mm_D2.5mm_P2.54mm_Vertical
- R14: footprint Resistor_THT:R_Axial_DIN0207_L6.3mm_D2.5mm_P7.62mm_Horizontal -> Resistor_THT:R_Axial_DIN0207_L6.3mm_D2.5mm_P2.54mm_Vertical
- R5: value 4.7K -> 10k
- R7: footprint Resistor_THT:R_Axial_DIN0204_L3.6mm_D1.6mm_P5.08mm_Horizontal -> Resistor_THT:R_Axial_DIN0207_L6.3mm_D2.5mm_P7.62mm_Horizontal
- R9: footprint Resistor_THT:R_Axial_DIN0207_L6.3mm_D2.5mm_P7.62mm_Horizontal -> Resistor_THT:R_Axial_DIN0204_L3.6mm_D1.6mm_P2.54mm_Vertical
- moved P3 93.3 mm to (38.7, 45.1), turned to 90 degrees
- moved P4 93.3 mm to (38.7, 37.5), turned to 90 degrees
- moved D4 86.2 mm to (48.3, 41.9), turned to 180 degrees
- moved J3 85.1 mm to (35.6, 55.2), turned to 180 degrees
- moved D6 83.8 mm to (48.3, 45.1), turned to 180 degrees
- moved R5 80.9 mm to (36.8, 62.2)
- moved D3 78.1 mm to (51.4, 48.9), turned to 90 degrees
- moved R12 77.5 mm to (48.3, 48.9), turned to 180 degrees
- moved R10 76.9 mm to (36.8, 59.1), turned to 0 degrees
- moved D7 73.1 mm to (45.7, 35.6), turned to 0 degrees
- moved D5 70.1 mm to (45.7, 38.7), turned to 0 degrees
- moved R13 70.0 mm to (43.2, 48.9), turned to 180 degrees
- moved R11 69.5 mm to (44.5, 61.6), turned to 0 degrees
- moved R9 52.8 mm to (59.1, 59.7), turned to 90 degrees
- moved R14 50.8 mm to (53.3, 33.0), turned to 0 degrees
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Connections:
- D2 pad 2: +5.0V -> Net-(D2-Pad2)
- J1 pad 1: +3.3V -> +5.0V
- J1 pad 10: PRI_RXD -> (no net)
- J1 pad 13: (no net) -> GNDREF
- J1 pad 14: GNDREF -> (no net)
- J1 pad 18: TEMP_INS -> (no net)
- J1 pad 19: (no net) -> GNDREF
- J1 pad 2: +5.0V -> +3.3V
- J1 pad 20: GNDREF -> (no net)
- J1 pad 24: (no net) -> TEMP_INS
- J1 pad 25: GNDREF -> (no net)
- J1 pad 26: (no net) -> GNDREF
- J1 pad 5: (no net) -> GNDREF
- J1 pad 6: GNDREF -> (no net)
- J1 pad 7: (no net) -> PRI_TXD
- J1 pad 8: PRI_TXD -> (no net)
- J1 pad 9: (no net) -> PRI_RXD
- P4 pad 1: Net-(D6-Pad2) -> Net-(D4-Pad2)
- P4 pad 2: Net-(D4-Pad2) -> Net-(D6-Pad2)
- Q1 pad 1: Net-(Q1-Pad1) -> Net-(D3-Pad2)
- R7 pad 1: Net-(R7-Pad1) -> Net-(D2-Pad2)
- R7 pad 2: Net-(D2-Pad1) -> +5.0V
- U2 pad 5: Net-(R7-Pad1) -> Net-(D2-Pad1)
Routing:
- net PRI_TXD: track 12.3 -> 68.0 mm
- net PRI_RXD: track 39.8 -> 82.8 mm
- net GNDREF: track 164.3 -> 126.4 mm
- net Net-(IC1-Pad2): track 37.3 -> 10.8 mm
- net Net-(D4-Pad2): track 46.5 -> 23.6 mm
- net +3.3V: track 25.4 -> 15.9 mm
- net Net-(R4-Pad1): track 3.05 -> 12.0 mm
- net Net-(D2-Pad1): track 3.18 -> 11.4 mm
- net Net-(D3-Pad2): track 14.0 -> 6.13 mm
- net Net-(D6-Pad2): track 27.7 -> 35.4 mm
- net Net-(IC1-Pad3): track 30.8 -> 23.1 mm
- net TEMP_INS: track 52.4 -> 58.5 mm, vias 0 -> 1
- net Net-(R6-Pad1): track 2.54 -> 8.04 mm
- net Net-(Q1-Pad2): track 21.1 -> 15.8 mm
- net Net-(R7-Pad1): track 4.45 -> 0.00 mm
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- added copper zone on B.Cu, net (none)
- added copper zone on F.Cu, net (none)
Other:
- board outline added: 50.8 x 38.7 mm
