File: adapter/ebus-pri.sch (KiCad schematic (older format))
At the start: 29 parts, among them IC1 TLC393CP, J1 Conn_02x13_Odd_Even, J3 DS18B20_IN, P3 ebus1, P4 ebus2, Q1 BC338, U1 CNY17-4, U2 CNY17-4

Commit message: ready for print
Parts:
- removed R15: 0ohm, Resistor_THT:R_Axial_DIN0207_L6.3mm_D2.5mm_P7.62mm_Horizontal, symbol Device:R
- D3: footprint Diode_THT:D_DO-41_SOD81_P12.70mm_Horizontal -> Diode_THT:D_DO-41_SOD81_P2.54mm_Vertical_KathodeUp
- D4, D5, D6, D7: footprint Diode_THT:D_DO-41_SOD81_P7.62mm_Horizontal -> Diode_THT:D_DO-41_SOD81_P2.54mm_Vertical_KathodeUp
- R11: footprint Resistor_THT:R_Axial_DIN0207_L6.3mm_D2.5mm_P10.16mm_Horizontal -> Resistor_THT:R_Axial_DIN0204_L3.6mm_D1.6mm_P2.54mm_Vertical
- R12: footprint Resistor_THT:R_Axial_DIN0309_L9.0mm_D3.2mm_P12.70mm_Horizontal -> Resistor_THT:R_Axial_DIN0207_L6.3mm_D2.5mm_P2.54mm_Vertical
- R13: footprint Resistor_THT:R_Axial_DIN0207_L6.3mm_D2.5mm_P10.16mm_Horizontal -> Resistor_THT:R_Axial_DIN0207_L6.3mm_D2.5mm_P2.54mm_Vertical
- R14: footprint Resistor_THT:R_Axial_DIN0207_L6.3mm_D2.5mm_P7.62mm_Horizontal -> Resistor_THT:R_Axial_DIN0207_L6.3mm_D2.5mm_P2.54mm_Vertical
- R5: value 4.7K -> 10k
- R7: footprint Resistor_THT:R_Axial_DIN0204_L3.6mm_D1.6mm_P5.08mm_Horizontal -> Resistor_THT:R_Axial_DIN0207_L6.3mm_D2.5mm_P7.62mm_Horizontal
- R9: footprint Resistor_THT:R_Axial_DIN0207_L6.3mm_D2.5mm_P7.62mm_Horizontal -> Resistor_THT:R_Axial_DIN0204_L3.6mm_D1.6mm_P2.54mm_Vertical
Connections:
- net +3.3V: now also J1.2 (Pin_2); no longer J1.1 (Pin_1)
- net +5.0V: now also J1.1 (Pin_1), R7.2; no longer D2.2 (A), J1.2 (Pin_2)
- net GNDREF: now also J1.13 (Pin_13), J1.19 (Pin_19), J1.26 (Pin_26), J1.5 (Pin_5); no longer J1.14 (Pin_14), J1.20 (Pin_20), J1.25 (Pin_25), J1.6 (Pin_6)
- net PRI_RXD: now also J1.9 (Pin_9); no longer J1.10 (Pin_10)
- net PRI_TXD: now also J1.7 (Pin_7); no longer J1.8 (Pin_8)
- net TEMP_INS: now also J1.17 (Pin_17); no longer J1.18 (Pin_18)
- net at D2.1 (K): now also U2.5; no longer R7.2
- net at R7.1: now also D2.2 (A); no longer U2.5
- net at D4.2 (A), D5.1 (K), P3.2 (Pin_2): now also P4.1 (Pin_1); no longer P4.2 (Pin_2)
- net at D3.2 (A): now also Q1.1 (C)
- net at D6.2 (A), D7.1 (K), P3.1 (Pin_1): now also P4.2 (Pin_2); no longer P4.1 (Pin_1)
Other:
- moved on the sheet: D2, R7
Changed lines of the file:
@@
 L Device:LED D2
 U 1 1 5D8907FF
+P 5900 4500
+F 0 "D2" H 5900 4600 50  0000 C CNN
+F 1 "LED TX" H 5900 4400 50  0000 C CNN
+F 2 "LED_THT:LED_D3.0mm" H 5900 4500 50  0001 C CNN
+F 3 "" H 5900 4500 50  0000 C CNN
+	1    5900 4500
+	0    -1   -1   0
+$EndComp
+$Comp
+L Device:R R7
+U 1 1 5D8908EA
 P 5900 4100
-F 0 "D2" H 5900 4200 50  0000 C CNN
-F 1 "LED TX" H 5900 4000 50  0000 C CNN
-F 2 "LED_THT:LED_D3.0mm" H 5900 4100 50  0001 C CNN
+F 0 "R7" V 5980 4100 50  0000 C CNN
+F 1 "470" V 5900 4100 50  0000 C CNN
+F 2 "Resistor_THT:R_Axial_DIN0207_L6.3mm_D2.5mm_P7.62mm_Horizontal" V 5830 4100 50  0001 C CNN
 F 3 "" H 5900 4100 50  0000 C CNN
 	1    5900 4100
-	0    -1   -1   0
-$EndComp
-$Comp
-L Device:R R7
-U 1 1 5D8908EA
-P 5900 4500
-F 0 "R7" V 5980 4500 50  0000 C CNN
-F 1 "470" V 5900 4500 50  0000 C CNN
-F 2 "Resistor_THT:R_Axial_DIN0204_L3.6mm_D1.6mm_P5.08mm_Horizontal" V 5830 4500 50  0001 C CNN
-F 3 "" H 5900 4500 50  0000 C CNN
-	1    5900 4500
 	1    0    0    1
 $EndComp
@@
 F 0 "R9" V 7780 3800 50  0000 C CNN
 F 1 "220K" V 7700 3800 50  0000 C CNN
-F 2 "Resistor_THT:R_Axial_DIN0207_L6.3mm_D2.5mm_P7.62mm_Horizontal" V 7630 3800 50  0001 C CNN
+F 2 "Resistor_THT:R_Axial_DIN0204_L3.6mm_D1.6mm_P2.54mm_Vertical" V 7630 3800 50  0001 C CNN
 F 3 "" H 7700 3800 50  0000 C CNN
 	1    7700 3800
@@
 F 0 "R11" V 8030 4950 50  0000 C CNN
 F 1 "15k" V 7950 4950 50  0000 C CNN
-F 2 "Resistor_THT:R_Axial_DIN0207_L6.3mm_D2.5mm_P10.16mm_Horizontal" V 7880 4950 50  0001 C CNN
+F 2 "Resistor_THT:R_Axial_DIN0204_L3.6mm_D1.6mm_P2.54mm_Vertical" V 7880 4950 50  0001 C CNN
 F 3 "" H 7950 4950 50  0000 C CNN
 	1    7950 4950
@@
 F 0 "R13" V 8430 4950 50  0000 C CNN
 F 1 "22k" V 8350 4950 50  0000 C CNN
-F 2 "Resistor_THT:R_Axial_DIN0207_L6.3mm_D2.5mm_P10.16mm_Horizontal" V 8280 4950 50  0001 C CNN
+F 2 "Resistor_THT:R_Axial_DIN0207_L6.3mm_D2.5mm_P2.54mm_Vertical" V 8280 4950 50  0001 C CNN
 F 3 "" H 8350 4950 50  0000 C CNN
 	1    8350 4950
@@
 F 0 "R12" V 8430 3450 50  0000 C CNN
 F 1 "100k" V 8350 3450 50  0000 C CNN
-F 2 "Resistor_THT:R_Axial_DIN0309_L9.0mm_D3.2mm_P12.70mm_Horizontal" V 8280 3450 50  0001 C CNN
+F 2 "Resistor_THT:R_Axial_DIN0207_L6.3mm_D2.5mm_P2.54mm_Vertical" V 8280 3450 50  0001 C CNN
 F 3 "" H 8350 3450 50  0000 C CNN
 	1    8350 3450
@@
 F 0 "D4" H 9450 4000 50  0000 C CNN
 F 1 "1N4007" H 9450 3800 50  0000 C CNN
-F 2 "Diode_THT:D_DO-41_SOD81_P7.62mm_Horizontal" H 9450 3725 50  0001 C CNN
+F 2 "Diode_THT:D_DO-41_SOD81_P2.54mm_Vertical_KathodeUp" H 9450 3725 50  0001 C CNN
 F 3 "" H 9450 3900 50  0001 C CNN
 	1    9450 3900
@@
 F 0 "D3" H 8850 4000 50  0000 C CNN
 F 1 "ZPY 9.1V 1.3W" H 8850 3800 50  0000 C CNN
-F 2 "Diode_THT:D_DO-41_SOD81_P12.70mm_Horizontal" H 8850 3900 50  0001 C CNN
+F 2 "Diode_THT:D_DO-41_SOD81_P2.54mm_Vertical_KathodeUp" H 8850 3900 50  0001 C CNN
 F 3 "" H 8850 3900 50  0001 C CNN
 	1    8850 3900
@@
 F 0 "D5" H 9450 4800 50  0000 C CNN
 F 1 "1N4007" H 9450 4600 50  0000 C CNN
-F 2 "Diode_THT:D_DO-41_SOD81_P7.62mm_Horizontal" H 9450 4525 50  0001 C CNN
+F 2 "Diode_THT:D_DO-41_SOD81_P2.54mm_Vertical_KathodeUp" H 9450 4525 50  0001 C CNN
 F 3 "" H 9450 4700 50  0001 C CNN
 	1    9450 4700
@@
 F 0 "D6" H 9900 4000 50  0000 C CNN
 F 1 "1N4007" H 9900 3800 50  0000 C CNN
-F 2 "Diode_THT:D_DO-41_SOD81_P7.62mm_Horizontal" H 9900 3725 50  0001 C CNN
+F 2 "Diode_THT:D_DO-41_SOD81_P2.54mm_Vertical_KathodeUp" H 9900 3725 50  0001 C CNN
 F 3 "" H 9900 3900 50  0001 C CNN
 	1    9900 3900
@@
 F 0 "D7" H 9900 4800 50  0000 C CNN
 F 1 "1N4007" H 9900 4600 50  0000 C CNN
-F 2 "Diode_THT:D_DO-41_SOD81_P7.62mm_Horizontal" H 9900 4525 50  0001 C CNN
+F 2 "Diode_THT:D_DO-41_SOD81_P2.54mm_Vertical_KathodeUp" H 9900 4525 50  0001 C CNN
 F 3 "" H 9900 4700 50  0001 C CNN
 	1    9900 4700
@@
 L Connector_Generic:Conn_01x02 P4
 U 1 1 5D893003
-P 10550 4550
-F 0 "P4" H 10550 4700 50  0000 C CNN
-F 1 "ebus2" V 10650 4550 50  0000 C CNN
-F 2 "Connector:JWT_A3963_1x02_P3.96mm_Vertical" H 10550 4550 50  0001 C CNN
-F 3 "" H 10550 4550 50  0000 C CNN
-	1    10550 4550
-	1    0    0    -1
+P 10550 4650
+F 0 "P4" H 10550 4800 50  0000 C CNN
+F 1 "ebus2" V 10650 4650 50  0000 C CNN
+F 2 "Connector:JWT_A3963_1x02_P3.96mm_Vertical" H 10550 4650 50  0001 C CNN
+F 3 "" H 10550 4650 50  0000 C CNN
+	1    10550 4650
+	1    0    0    1
 $EndComp
 $Comp
@@
 F 0 "R14" V 8580 5850 50  0000 C CNN
 F 1 "220" V 8500 5850 50  0000 C CNN
-F 2 "Resistor_THT:R_Axial_DIN0207_L6.3mm_D2.5mm_P7.62mm_Horizontal" V 8430 5850 50  0001 C CNN
+F 2 "Resistor_THT:R_Axial_DIN0207_L6.3mm_D2.5mm_P2.54mm_Vertical" V 8430 5850 50  0001 C CNN
 F 3 "" H 8500 5850 50  0001 C CNN
 	1    8500 5850
@@
 P 4850 1100
 F 0 "R5" V 4930 1100 50  0000 C CNN
-F 1 "4.7K" V 4850 1100 50  0000 C CNN
+F 1 "10k" V 4850 1100 50  0000 C CNN
 F 2 "Resistor_THT:R_Axial_DIN0204_L3.6mm_D1.6mm_P2.54mm_Vertical" V 4780 1100 50  0001 C CNN
 F 3 "" H 4850 1100 50  0001 C CNN
@@
 +5.0V
 Wire Wire Line
-	2950 5550 3100 5550
-Wire Wire Line
 	2300 6800 2300 6750
-Wire Wire Line
-	2300 6750 2450 6750
-Wire Wire Line
-	2950 5850 3100 5850
-Wire Wire Line
-	2950 5950 3100 5950
-Wire Wire Line
-	2950 6350 3100 6350
 $Comp
 L Connector_Generic:Conn_01x03 J3
@@
 	1    0    0    -1
 $EndComp
-$Comp
-L Connector_Generic:Conn_02x13_Odd_Even J1
-U 1 1 5D9A85EF
-P 2650 6150
-F 0 "J1" H 2700 6967 50  0000 C CNN
-F 1 "Conn_02x13_Odd_Even" H 2700 6876 50  0000 C CNN
-F 2 "Connector_PinHeader_2.54mm:PinHeader_2x13_P2.54mm_Vertical" H 2650 6150 50  0001 C CNN
-F 3 "~" H 2650 6150 50  0001 C CNN
-	1    2650 6150
-	1    0    0    -1
-$EndComp
 Wire Wire Line
 	9650 5000 9650 5150
-Wire Wire Line
-	2950 5750 3800 5750
 $Comp
 L power:GNDREF #PWR010
@@
 $EndComp
 Wire Wire Line
-	2950 6150 3800 6150
-Wire Wire Line
 	3800 5750 3800 6150
 Connection ~ 3800 6150
-Wire Wire Line
-	2950 6450 3800 6450
 Wire Wire Line
 	3800 6150 3800 6450
@@
 Text GLabel 2150 5550 0    50   Input ~ 0
 +3.3V
-Wire Wire Line
-	2450 5550 2150 5550
 Text GLabel 4450 4400 1    50   Input ~ 0
 +3.3V
@@
 $EndComp
 $Comp
-L Device:R R15
-U 1 1 5DFE511C
-P 8850 4650
-F 0 "R15" V 8930 4650 50  0000 C CNN
-F 1 "0ohm" V 8850 4650 50  0000 C CNN
-F 2 "Resistor_THT:R_Axial_DIN0207_L6.3mm_D2.5mm_P7.62mm_Horizontal" V 8780 4650 50  0001 C CNN
-F 3 "" H 8850 4650 50  0000 C CNN
-	1    8850 4650
-	-1   0    0    1
-$EndComp
-Wire Wire Line
-	8850 4050 8850 4500
-Wire Wire Line
-	8850 4800 8850 5350
+L Connector_Generic:Conn_02x13_Odd_Even J1
+U 1 1 5D9A85EF
+P 2750 6150
+F 0 "J1" H 2800 6967 50  0000 C CNN
+F 1 "Conn_02x13_Odd_Even" H 2800 6876 50  0000 C CNN
+F 2 "Connector_PinHeader_2.54mm:PinHeader_2x13_P2.54mm_Vertical" H 2750 6150 50  0001 C CNN
+F 3 "~" H 2750 6150 50  0001 C CNN
+	1    2750 6150
+	-1   0    0    -1
+$EndComp
+Wire Wire Line
+	2950 5550 3100 5550
+Wire Wire Line
+	2950 5950 3100 5950
+Wire Wire Line
+	2950 5750 3800 5750
+Wire Wire Line
+	2950 6150 3800 6150
+Wire Wire Line
+	2950 6450 3800 6450
+Wire Wire Line
+	2300 6750 2450 6750
+Wire Wire Line
+	2150 5550 2450 5550
+Wire Wire Line
+	2950 5850 3100 5850
+Wire Wire Line
+	2950 6350 3100 6350
+Wire Wire Line
+	8850 4050 8850 5350
 $EndSCHEMATC
